Commit message: making all finger and multisense joints fixed for a planning urdf

File: model/robots/common/xacro/index_finger/index_finger.xacro (robot description, xacro)
@@ -32,40 +32,19 @@
                     visual_mesh="${mesh_root}/fingers/indexj3_${prefix}.dae"
                     collision_mesh="${mesh_root}/fingers/indexj3_${prefix}.dae"/>
-    <xacro:revolute_joint jointName="${IndexFingerPitch1JointName}"
+    <xacro:fixed_joint jointName="${IndexFingerPitch1JointName}"
                           parent="${IndexFingerPitch1ParentLinkName}" child="${IndexFingerPitch1LinkName}"
                           origin_xyz="${IndexFingerPitch1FrameOrigin_X} ${IndexFingerPitch1FrameOrigin_Y} ${IndexFingerPitch1FrameOrigin_Z}"
-                          origin_rpy="${IndexFingerPitch1FrameOrientation_Roll} ${IndexFingerPitch1FrameOrientation_Pitch} ${IndexFingerPitch1FrameOrientation_Yaw}"
-                          axis="${IndexFingerPitch1RotationAxis}">
-        <xacro:if value="${(reflect+1)/2}">
-          <limit effort="${IndexFingerPitch1TorqueLimit}" lower="${-reflect * IndexFingerPitch1PositionLimit_Upper}" upper="${-reflect * IndexFingerPitch1PositionLimit_Lower}" velocity="${IndexFingerPitch1VelocityLimit}"/>
-        </xacro:if>
-        <xacro:if value="${(-reflect+1)/2}">
-          <limit effort="${IndexFingerPitch1TorqueLimit}" lower="${IndexFingerPitch1PositionLimit_Lower}" upper="${IndexFingerPitch1PositionLimit_Upper}" velocity="${IndexFingerPitch1VelocityLimit}"/>
-        </xacro:if>
-    </xacro:revolute_joint>
-    <xacro:revolute_joint jointName="${IndexFingerPitch2JointName}"
+                          origin_rpy="${IndexFingerPitch1FrameOrientation_Roll} ${IndexFingerPitch1FrameOrientation_Pitch} ${IndexFingerPitch1FrameOrientation_Yaw}">
+    </xacro:fixed_joint>
+    <xacro:fixed_joint jointName="${IndexFingerPitch2JointName}"
                           parent="${IndexFingerPitch1LinkName}" child="${IndexFingerPitch2LinkName}"
                           origin_xyz="${IndexFingerPitch2FrameOrigin_X} ${IndexFingerPitch2FrameOrigin_Y} ${IndexFingerPitch2FrameOrigin_Z}"
-                          origin_rpy="${IndexFingerPitch2FrameOrientation_Roll} ${IndexFingerPitch2FrameOrientation_Pitch} ${IndexFingerPitch2FrameOrientation_Yaw}"
-                          axis="${IndexFingerPitch2RotationAxis}">
-        <xacro:if value="${(reflect+1)/2}">
-          <limit effort="${IndexFingerPitch2TorqueLimit}" lower="${-reflect * IndexFingerPitch2PositionLimit_Upper}" upper="${-reflect * IndexFingerPitch2PositionLimit_Lower}" velocity="${IndexFingerPitch2VelocityLimit}"/>
-        </xacro:if>
-        <xacro:if value="${(-reflect+1)/2}">
-          <limit effort="${IndexFingerPitch2TorqueLimit}" lower="${IndexFingerPitch2PositionLimit_Lower}" upper="${IndexFingerPitch2PositionLimit_Upper}" velocity="${IndexFingerPitch2VelocityLimit}"/>
-        </xacro:if>
-    </xacro:revolute_joint>
-    <xacro:revolute_joint jointName="${IndexFingerPitch3JointName}"
+                          origin_rpy="${IndexFingerPitch2FrameOrientation_Roll} ${IndexFingerPitch2FrameOrientation_Pitch} ${IndexFingerPitch2FrameOrientation_Yaw}">
+    </xacro:fixed_joint>
+    <xacro:fixed_joint jointName="${IndexFingerPitch3JointName}"
                           parent="${IndexFingerPitch2LinkName}" child="${IndexFingerPitch3LinkName}"
                           origin_xyz="${IndexFingerPitch3FrameOrigin_X} ${IndexFingerPitch3FrameOrigin_Y} ${IndexFingerPitch3FrameOrigin_Z}"
-                          origin_rpy="${IndexFingerPitch3FrameOrientation_Roll} ${IndexFingerPitch3FrameOrientation_Pitch} ${IndexFingerPitch3FrameOrientation_Yaw}"
-                          axis="${IndexFingerPitch3RotationAxis}">
-        <xacro:if value="${(reflect+1)/2}">
-          <limit effort="${IndexFingerPitch3TorqueLimit}" lower="${-reflect * IndexFingerPitch3PositionLimit_Upper}" upper="${-reflect * IndexFingerPitch3PositionLimit_Lower}" velocity="${IndexFingerPitch3VelocityLimit}"/>
-        </xacro:if>
-        <xacro:if value="${(-reflect+1)/2}">
-          <limit effort="${IndexFingerPitch3TorqueLimit}" lower="${IndexFingerPitch3PositionLimit_Lower}" upper="${IndexFingerPitch3PositionLimit_Upper}" velocity="${IndexFingerPitch3VelocityLimit}"/>
-        </xacro:if>
-    </xacro:revolute_joint>
+                          origin_rpy="${IndexFingerPitch3FrameOrientation_Roll} ${IndexFingerPitch3FrameOrientation_Pitch} ${IndexFingerPitch3FrameOrientation_Yaw}">
+    </xacro:fixed_joint>
   </xacro:macro>
   <xacro:macro name="index_finger_transmissions_hw" params="prefix">

File: model/robots/common/xacro/middle_finger/middle_finger.xacro (robot description, xacro)
@@ -32,40 +32,19 @@
                     visual_mesh="${mesh_root}/fingers/middlej3_${prefix}.dae"
                     collision_mesh="${mesh_root}/fingers/middlej3_${prefix}.dae"/>
-    <xacro:revolute_joint jointName="${MiddleFingerPitch1JointName}"
+    <xacro:fixed_joint jointName="${MiddleFingerPitch1JointName}"
                           parent="${MiddleFingerPitch1ParentLinkName}" child="${MiddleFingerPitch1LinkName}"
                           origin_xyz="${MiddleFingerPitch1FrameOrigin_X} ${MiddleFingerPitch1FrameOrigin_Y} ${MiddleFingerPitch1FrameOrigin_Z}"
-                          origin_rpy="${MiddleFingerPitch1FrameOrientation_Roll} ${MiddleFingerPitch1FrameOrientation_Pitch} ${MiddleFingerPitch1FrameOrientation_Yaw}"
-                          axis="${MiddleFingerPitch1RotationAxis}">
-        <xacro:if value="${(reflect+1)/2}">
-          <limit effort="${MiddleFingerPitch1TorqueLimit}" lower="${-reflect * MiddleFingerPitch1PositionLimit_Upper}" upper="${-reflect * MiddleFingerPitch1PositionLimit_Lower}" velocity="${MiddleFingerPitch1VelocityLimit}"/>
-        </xacro:if>
-        <xacro:if value="${(-reflect+1)/2}">
-          <limit effort="${MiddleFingerPitch1TorqueLimit}" lower="${MiddleFingerPitch1PositionLimit_Lower}" upper="${MiddleFingerPitch1PositionLimit_Upper}" velocity="${MiddleFingerPitch1VelocityLimit}"/>
-        </xacro:if>
-    </xacro:revolute_joint>
-    <xacro:revolute_joint jointName="${MiddleFingerPitch2JointName}"
+                          origin_rpy="${MiddleFingerPitch1FrameOrientation_Roll} ${MiddleFingerPitch1FrameOrientation_Pitch} ${MiddleFingerPitch1FrameOrientation_Yaw}">
+    </xacro:fixed_joint>
+    <xacro:fixed_joint jointName="${MiddleFingerPitch2JointName}"
                           parent="${MiddleFingerPitch1LinkName}" child="${MiddleFingerPitch2LinkName}"
                           origin_xyz="${MiddleFingerPitch2FrameOrigin_X} ${MiddleFingerPitch2FrameOrigin_Y} ${MiddleFingerPitch2FrameOrigin_Z}"
-                          origin_rpy="${MiddleFingerPitch2FrameOrientation_Roll} ${MiddleFingerPitch2FrameOrientation_Pitch} ${MiddleFingerPitch2FrameOrientation_Yaw}"
-                          axis="${MiddleFingerPitch2RotationAxis}">
-        <xacro:if value="${(reflect+1)/2}">
-          <limit effort="${MiddleFingerPitch2TorqueLimit}" lower="${-reflect * MiddleFingerPitch2PositionLimit_Upper}" upper="${-reflect * MiddleFingerPitch2PositionLimit_Lower}" velocity="${MiddleFingerPitch2VelocityLimit}"/>
-        </xacro:if>
-        <xacro:if value="${(-reflect+1)/2}">
-          <limit effort="${MiddleFingerPitch2TorqueLimit}" lower="${MiddleFingerPitch2PositionLimit_Lower}" upper="${MiddleFingerPitch2PositionLimit_Upper}" velocity="${MiddleFingerPitch2VelocityLimit}"/>
-        </xacro:if>
-    </xacro:revolute_joint>
-    <xacro:revolute_joint jointName="${MiddleFingerPitch3JointName}"
+                          origin_rpy="${MiddleFingerPitch2FrameOrientation_Roll} ${MiddleFingerPitch2FrameOrientation_Pitch} ${MiddleFingerPitch2FrameOrientation_Yaw}">
+    </xacro:fixed_joint>
+    <xacro:fixed_joint jointName="${MiddleFingerPitch3JointName}"
                           parent="${MiddleFingerPitch2LinkName}" child="${MiddleFingerPitch3LinkName}"
                           origin_xyz="${MiddleFingerPitch3FrameOrigin_X} ${MiddleFingerPitch3FrameOrigin_Y} ${MiddleFingerPitch3FrameOrigin_Z}"
-                          origin_rpy="${MiddleFingerPitch3FrameOrientation_Roll} ${MiddleFingerPitch3FrameOrientation_Pitch} ${MiddleFingerPitch3FrameOrientation_Yaw}"
-                          axis="${MiddleFingerPitch3RotationAxis}">
-        <xacro:if value="${(reflect+1)/2}">
-          <limit effort="${MiddleFingerPitch3TorqueLimit}" lower="${-reflect * MiddleFingerPitch3PositionLimit_Upper}" upper="${-reflect * MiddleFingerPitch3PositionLimit_Lower}" velocity="${MiddleFingerPitch3VelocityLimit}"/>
-        </xacro:if>
-        <xacro:if value="${(-reflect+1)/2}">
-          <limit effort="${MiddleFingerPitch3TorqueLimit}" lower="${MiddleFingerPitch3PositionLimit_Lower}" upper="${MiddleFingerPitch3PositionLimit_Upper}" velocity="${MiddleFingerPitch3VelocityLimit}"/>
-        </xacro:if>
-    </xacro:revolute_joint>
+                          origin_rpy="${MiddleFingerPitch3FrameOrientation_Roll} ${MiddleFingerPitch3FrameOrientation_Pitch} ${MiddleFingerPitch3FrameOrientation_Yaw}">
+    </xacro:fixed_joint>
   </xacro:macro>
   <xacro:macro name="middle_finger_transmissions_hw" params="prefix">

File: model/robots/common/xacro/pinky_finger/pinky_finger.xacro (robot description, xacro)
@@ -32,40 +32,20 @@
                     visual_mesh="${mesh_root}/fingers/pinkyj3_${prefix}.dae"
                     collision_mesh="${mesh_root}/fingers/pinkyj3_${prefix}.dae"/>
-    <xacro:revolute_joint jointName="${PinkyPitch1JointName}"
+    <xacro:fixed_joint jointName="${PinkyPitch1JointName}"
                           parent="${PinkyPitch1ParentLinkName}" child="${PinkyPitch1LinkName}"
                           origin_xyz="${PinkyPitch1FrameOrigin_X} ${PinkyPitch1FrameOrigin_Y} ${PinkyPitch1FrameOrigin_Z}"
-                          origin_rpy="${PinkyPitch1FrameOrientation_Roll} ${PinkyPitch1FrameOrientation_Pitch} ${PinkyPitch1FrameOrientation_Yaw}"
-                          axis="${PinkyFingerPitch1RotationAxis}">
-        <xacro:if value="${(reflect+1)/2}">
-          <limit effort="${PinkyFingerPitch1TorqueLimit}" lower="${-reflect * PinkyFingerPitch1PositionLimit_Upper}" upper="${-reflect * PinkyFingerPitch1PositionLimit_Lower}" velocity="${PinkyFingerPitch1VelocityLimit}"/>
-        </xacro:if>
-        <xacro:if value="${(-reflect+1)/2}">
-          <limit effort="${PinkyFingerPitch1TorqueLimit}" lower="${PinkyFingerPitch1PositionLimit_Lower}" upper="${PinkyFingerPitch1PositionLimit_Upper}" velocity="${PinkyFingerPitch1VelocityLimit}"/>
-        </xacro:if>
-    </xacro:revolute_joint>
-    <xacro:revolute_joint jointName="${PinkyPitch2JointName}"
+                          origin_rpy="${PinkyPitch1FrameOrientation_Roll} ${PinkyPitch1FrameOrientation_Pitch} ${PinkyPitch1FrameOrientation_Yaw}">
+        <limit effort="${PinkyPitch1TorqueLimit}" lower="${PinkyPitch1PositionLimit_Lower}" upper="${PinkyPitch1PositionLimit_Upper}" velocity="${PinkyPitch1VelocityLimit}"/>
+    </xacro:fixed_joint>
+    <xacro:fixed_joint jointName="${PinkyPitch2JointName}"
                           parent="${PinkyPitch1LinkName}" child="${PinkyPitch2LinkName}"
                           origin_xyz="${PinkyPitch2FrameOrigin_X} ${PinkyPitch2FrameOrigin_Y} ${PinkyPitch2FrameOrigin_Z}"
-                          origin_rpy="${PinkyPitch2FrameOrientation_Roll} ${PinkyPitch2FrameOrientation_Pitch} ${PinkyPitch2FrameOrientation_Yaw}"
-                          axis="${PinkyFingerPitch2RotationAxis}">
-        <xacro:if value="${(reflect+1)/2}">
-          <limit effort="${PinkyFingerPitch2TorqueLimit}" lower="${-reflect * PinkyFingerPitch2PositionLimit_Upper}" upper="${-reflect * PinkyFingerPitch2PositionLimit_Lower}" velocity="${PinkyFingerPitch2VelocityLimit}"/>
-        </xacro:if>
-        <xacro:if value="${(-reflect+1)/2}">
-          <limit effort="${PinkyFingerPitch2TorqueLimit}" lower="${PinkyFingerPitch2PositionLimit_Lower}" upper="${PinkyFingerPitch2PositionLimit_Upper}" velocity="${PinkyFingerPitch2VelocityLimit}"/>
-        </xacro:if>
-    </xacro:revolute_joint>
-    <xacro:revolute_joint jointName="${PinkyPitch3JointName}"
+                          origin_rpy="${PinkyPitch2FrameOrientation_Roll} ${PinkyPitch2FrameOrientation_Pitch} ${PinkyPitch2FrameOrientation_Yaw}">
+    </xacro:fixed_joint>
+    <xacro:fixed_joint jointName="${PinkyPitch3JointName}"
                           parent="${PinkyPitch2LinkName}" child="${PinkyPitch3LinkName}"
                           origin_xyz="${PinkyPitch3FrameOrigin_X} ${PinkyPitch3FrameOrigin_Y} ${PinkyPitch3FrameOrigin_Z}"
-                          origin_rpy="${PinkyPitch3FrameOrientation_Roll} ${PinkyPitch3FrameOrientation_Pitch} ${PinkyPitch3FrameOrientation_Yaw}"
-                          axis="${PinkyFingerPitch3RotationAxis}">
-        <xacro:if value="${(reflect+1)/2}">
-          <limit effort="${PinkyFingerPitch3TorqueLimit}" lower="${-reflect * PinkyFingerPitch3PositionLimit_Upper}" upper="${-reflect * PinkyFingerPitch3PositionLimit_Lower}" velocity="${PinkyFingerPitch3VelocityLimit}"/>
-        </xacro:if>
-        <xacro:if value="${(-reflect+1)/2}">
-          <limit effort="${PinkyFingerPitch3TorqueLimit}" lower="${PinkyFingerPitch3PositionLimit_Lower}" upper="${PinkyFingerPitch3PositionLimit_Upper}" velocity="${PinkyFingerPitch3VelocityLimit}"/>
-        </xacro:if>
-    </xacro:revolute_joint>
+                          origin_rpy="${PinkyPitch3FrameOrientation_Roll} ${PinkyPitch3FrameOrientation_Pitch} ${PinkyPitch3FrameOrientation_Yaw}">
+    </xacro:fixed_joint>
   </xacro:macro>
   <xacro:macro name="pinky_finger_transmissions_hw" params="prefix">

File: model/robots/common/xacro/thumb/thumb.xacro (robot description, xacro)
@@ -40,47 +40,24 @@
                     visual_mesh="${mesh_root}/fingers/thumbj4_${prefix}.dae"
                     collision_mesh="${mesh_root}/fingers/thumbj4_${prefix}.dae"/>
-    <xacro:revolute_joint jointName="${ThumbRollJointName}"
+    <xacro:fixed_joint jointName="${ThumbRollJointName}"
                           parent="${ThumbRollParentLinkName}" child="${ThumbRollLinkName}"
                           origin_xyz="${ThumbRollFrameOrigin_X} ${ThumbRollFrameOrigin_Y} ${ThumbRollFrameOrigin_Z}"
-                          origin_rpy="${ThumbRollFrameOrientation_Roll} ${ThumbRollFrameOrientation_Pitch} ${ThumbRollFrameOrientation_Yaw}"
-                          axis="${ThumbRollRotationAxis}">
-        <limit effort="${ThumbRollTorqueLimit}" lower="${ThumbRollPositionLimit_Lower}" upper="${ThumbRollPositionLimit_Upper}" velocity="${ThumbRollVelocityLimit}"/>
-    </xacro:revolute_joint>
-    <xacro:revolute_joint jointName="${ThumbPitch1JointName}"
+                          origin_rpy="${ThumbRollFrameOrientation_Roll} ${ThumbRollFrameOrientation_Pitch} ${ThumbRollFrameOrientation_Yaw}">
+    </xacro:fixed_joint>
+    <xacro:fixed_joint jointName="${ThumbPitch1JointName}"
                           parent="${ThumbRollLinkName}" child="${ThumbPitch1LinkName}"
                           origin_xyz="${ThumbPitch1FrameOrigin_X} ${ThumbPitch1FrameOrigin_Y} ${ThumbPitch1FrameOrigin_Z}"
-                          origin_rpy="${ThumbPitch1FrameOrientation_Roll} ${ThumbPitch1FrameOrientation_Pitch} ${ThumbPitch1FrameOrientation_Yaw}"
-                          axis="${ThumbPitch1RotationAxis}">
-        <xacro:if value="${(reflect+1)/2}">
-          <limit effort="${ThumbPitch1TorqueLimit}" lower="${-reflect * ThumbPitch1PositionLimit_Upper}" upper="${-reflect * ThumbPitch1PositionLimit_Lower}" velocity="${ThumbPitch1VelocityLimit}"/>
-        </xacro:if>
-        <xacro:if value="${(-reflect+1)/2}">
-          <limit effort="${ThumbPitch1TorqueLimit}" lower="${ThumbPitch1PositionLimit_Lower}" upper="${ThumbPitch1PositionLimit_Upper}" velocity="${ThumbPitch1VelocityLimit}"/>
-        </xacro:if>
-    </xacro:revolute_joint>
-    <xacro:revolute_joint jointName="${ThumbPitch2JointName}"
+                          origin_rpy="${ThumbPitch1FrameOrientation_Roll} ${ThumbPitch1FrameOrientation_Pitch} ${ThumbPitch1FrameOrientation_Yaw}">
+    </xacro:fixed_joint>
+    <xacro:fixed_joint jointName="${ThumbPitch2JointName}"
                           parent="${ThumbPitch1LinkName}" child="${ThumbPitch2LinkName}"
                           origin_xyz="${ThumbPitch2FrameOrigin_X} ${ThumbPitch2FrameOrigin_Y} ${ThumbPitch2FrameOrigin_Z}"
-                          origin_rpy="${ThumbPitch2FrameOrientation_Roll} ${ThumbPitch2FrameOrientation_Pitch} ${ThumbPitch2FrameOrientation_Yaw}"
-                          axis="${ThumbPitch2RotationAxis}">
-        <xacro:if value="${(reflect+1)/2}">
-          <limit effort="${ThumbPitch2TorqueLimit}" lower="${-reflect * ThumbPitch2PositionLimit_Upper}" upper="${-reflect * ThumbPitch2PositionLimit_Lower}" velocity="${ThumbPitch2VelocityLimit}"/>
-        </xacro:if>
-        <xacro:if value="${(-reflect+1)/2}">
-          <limit effort="${ThumbPitch2TorqueLimit}" lower="${ThumbPitch2PositionLimit_Lower}" upper="${ThumbPitch2PositionLimit_Upper}" velocity="${ThumbPitch2VelocityLimit}"/>
-        </xacro:if>
-    </xacro:revolute_joint>
-    <xacro:revolute_joint jointName="${ThumbPitch3JointName}"
+                          origin_rpy="${ThumbPitch2FrameOrientation_Roll} ${ThumbPitch2FrameOrientation_Pitch} ${ThumbPitch2FrameOrientation_Yaw}">
+    </xacro:fixed_joint>
+    <xacro:fixed_joint jointName="${ThumbPitch3JointName}"
                           parent="${ThumbPitch2LinkName}" child="${ThumbPitch3LinkName}"
                           origin_xyz="${ThumbPitch3FrameOrigin_X} ${ThumbPitch3FrameOrigin_Y} ${ThumbPitch3FrameOrigin_Z}"
-                          origin_rpy="${ThumbPitch3FrameOrientation_Roll} ${ThumbPitch3FrameOrientation_Pitch} ${ThumbPitch3FrameOrientation_Yaw}"
-                          axis="${ThumbPitch3RotationAxis}">
-        <xacro:if value="${(reflect+1)/2}">
-          <limit effort="${ThumbPitch3TorqueLimit}" lower="${-reflect * ThumbPitch3PositionLimit_Upper}" upper="${-reflect * ThumbPitch3PositionLimit_Lower}" velocity="${ThumbPitch3VelocityLimit}"/>
-        </xacro:if>
-        <xacro:if value="${(-reflect+1)/2}">
-          <limit effort="${ThumbPitch3TorqueLimit}" lower="${ThumbPitch3PositionLimit_Lower}" upper="${ThumbPitch3PositionLimit_Upper}" velocity="${ThumbPitch3VelocityLimit}"/>
-        </xacro:if>
-    </xacro:revolute_joint>
+                          origin_rpy="${ThumbPitch3FrameOrientation_Roll} ${ThumbPitch3FrameOrientation_Pitch} ${ThumbPitch3FrameOrientation_Yaw}">
+    </xacro:fixed_joint>
   </xacro:macro>
   <xacro:macro name="thumb_transmissions_hw" params="prefix">
