Commit message: move the hand goal frame to somewhere useful

File: model/robots/edinburgh_mods.xacro (robot description, xacro)
@@ -51,5 +51,5 @@
   </link>
   <joint name="l_hand_face_joint" type="fixed">
-    <origin rpy="3.14159265359 0 1.57079632679" xyz="0.07 0.0 -0.08"/>
+    <origin rpy="3.14159265359 0 1.57079632679" xyz="0.06 0.0 -0.045"/>
     <parent link="l_hand_force_torque"/>
     <child link="l_hand_face"/>
@@ -101,5 +101,5 @@
   </link>
   <joint name="r_hand_face_joint" type="fixed">
-    <origin rpy="0 0 -1.57079632679" xyz="0.07 0 0.08"/>
+    <origin rpy="0 0 -1.57079632679" xyz="0.06 0 0.045"/>
     <parent link="r_hand_force_torque"/>
     <child link="r_hand_face"/>
