Commit message: Fix gazebo force_torque sensors
Revert part of d17039f30ec944776c35a47a5e33ac6b218a4ade
to ensure that force_torque sensors are attached to ankle joints

File: model/robots/common/xacro/leg/leg.xacro (robot description, xacro)
@@ -154,4 +154,5 @@
     <xacro:ati_force_torque_sensor sensorName="${prefix}FootSixAxis"
                         parentLink="${AnkleRollLinkName}"
+                        joint_to_attach_sensor_to="${AnkleRollJointName}"
                         origin_xyz="0.0215646 0.0 -0.051054"
                         origin_rpy="3.14 0.0 0.0"

File: model/robots/common/xacro/sensors/ati_force_torque.xacro (robot description, xacro)
@@ -1,5 +1,5 @@
 <?xml version="1.0" ?>
 <robot xmlns:xacro="http://www.ros.org/wiki/xacro" name="ati_force_torque_sensor">
-  <xacro:macro name="ati_force_torque_sensor" params="sensorName parentLink origin_xyz origin_rpy sensor_number sensor_node sensor_api">
+  <xacro:macro name="ati_force_torque_sensor" params="sensorName parentLink joint_to_attach_sensor_to origin_xyz origin_rpy sensor_number sensor_node sensor_api">
     <xacro:massless_virtual_link name="${sensorName}_Frame"
                     origin_rpy="0 0 0"
@@ -9,7 +9,7 @@
                        origin_rpy="${origin_rpy}"
                        origin_xyz="${origin_xyz}"/>
-    <gazebo reference="${sensorName}_Frame">
+    <gazebo reference="${joint_to_attach_sensor_to}">
       <sensor name="${sensorName}" type="force_torque">
-        <pose>0 0 0 0 0 0 </pose>
+        <pose>${origin_xyz} ${origin_rpy}</pose>
         <sensor_number id="${sensor_number}" />
         <node id="${sensor_node}" />
