Commit message: Put unit A left leg on unit C, so switched relevant serial numbers.

File: common/xacro/serial_numbers/valkyrie_A_serials.xacro (robot description, xacro)
@@ -1,9 +1,9 @@
 <robot xmlns:xacro="http://ros.org/wiki/xacro" name="valkyrie_A_serials">
 	<xacro:property name="leftLegJ1SerialNumber" value="v_a_006" />
-	<xacro:property name="leftLegJ2SerialNumber" value="v_b_002" />
-	<xacro:property name="leftLegJ3SerialNumber" value="v_c_002" />
-	<xacro:property name="leftLegJ4SerialNumber" value="v_d_005" />
-	<xacro:property name="leftAnkleLeftActuatorSerialNumber" value="v_e_001" />
-	<xacro:property name="leftAnkleRightActuatorSerialNumber" value="v_e_002" />
+	<xacro:property name="leftLegJ2SerialNumber" value="v_b_006" />
+        <xacro:property name="leftLegJ3SerialNumber" value="v_c_004" />
+        <xacro:property name="leftLegJ4SerialNumber" value="v_d_003" />
+        <xacro:property name="leftAnkleLeftActuatorSerialNumber" value="v_e_019" />
+        <xacro:property name="leftAnkleRightActuatorSerialNumber" value="v_e_020" />
 	<xacro:property name="rightLegJ1SerialNumber" value="v_a_003" />
 	<xacro:property name="rightLegJ2SerialNumber" value="v_b_001" />
@@ -29,6 +29,6 @@
 	<xacro:property name="waistLeftActuatorSerialNumber" value="v_e_006" />
 	<xacro:property name="leftForearmSerialNumber" value="v_h_001"/>
-    <xacro:property name="rightForearmSerialNumber" value="v_h_002"/>
-	<xacro:property name="left_foot_ATI_serial" value="FT14020" />
+        <xacro:property name="rightForearmSerialNumber" value="v_h_002"/>
+	<xacro:property name="left_foot_ATI_serial" value="FT16594" />
 	<xacro:property name="right_foot_ATI_serial" value="FT16592" />
 	<xacro:property name="sim_ATI_serial" value="FT001SIM" />

File: common/xacro/serial_numbers/valkyrie_C_serials.xacro (robot description, xacro)
@@ -1,9 +1,9 @@
 <robot xmlns:xacro="http://ros.org/wiki/xacro" name="valkyrie_C_serials">
 	<xacro:property name="leftLegJ1SerialNumber" value="v_a_015" />
-	<xacro:property name="leftLegJ2SerialNumber" value="v_b_006" />
-    <xacro:property name="leftLegJ3SerialNumber" value="v_c_004" />
-    <xacro:property name="leftLegJ4SerialNumber" value="v_d_003" />
-    <xacro:property name="leftAnkleLeftActuatorSerialNumber" value="v_e_019" />
-    <xacro:property name="leftAnkleRightActuatorSerialNumber" value="v_e_020" />
+	<xacro:property name="leftLegJ2SerialNumber" value="v_b_002" />
+	<xacro:property name="leftLegJ3SerialNumber" value="v_c_002" />
+	<xacro:property name="leftLegJ4SerialNumber" value="v_d_005" />
+	<xacro:property name="leftAnkleLeftActuatorSerialNumber" value="v_e_001" />
+	<xacro:property name="leftAnkleRightActuatorSerialNumber" value="v_e_002" />
 	<xacro:property name="rightLegJ1SerialNumber" value="v_a_014" />
 	<xacro:property name="rightLegJ2SerialNumber" value="v_b_007" />
@@ -29,6 +29,6 @@
 	<xacro:property name="waistLeftActuatorSerialNumber" value="v_e_013" />
 	<xacro:property name="leftForearmSerialNumber" value="v_h_007"/>
-    <xacro:property name="rightForearmSerialNumber" value="v_h_008"/>
-	<xacro:property name="left_foot_ATI_serial" value="FT16594" />
+        <xacro:property name="rightForearmSerialNumber" value="v_h_008"/>
+	<xacro:property name="left_foot_ATI_serial" value="FT14020" />
 	<xacro:property name="right_foot_ATI_serial" value="FT17214" />
 	<xacro:property name="sim_ATI_serial" value="FT001SIM" />

Commit message: Swapped forearm coeff serial numbers.

File: common/xacro/serial_numbers/valkyrie_A_serials.xacro (robot description, xacro)
@@ -2,8 +2,8 @@
 	<xacro:property name="leftLegJ1SerialNumber" value="v_a_006" />
 	<xacro:property name="leftLegJ2SerialNumber" value="v_b_006" />
-        <xacro:property name="leftLegJ3SerialNumber" value="v_c_004" />
-        <xacro:property name="leftLegJ4SerialNumber" value="v_d_003" />
-        <xacro:property name="leftAnkleLeftActuatorSerialNumber" value="v_e_019" />
-        <xacro:property name="leftAnkleRightActuatorSerialNumber" value="v_e_020" />
+    <xacro:property name="leftLegJ3SerialNumber" value="v_c_004" />
+    <xacro:property name="leftLegJ4SerialNumber" value="v_d_003" />
+    <xacro:property name="leftAnkleLeftActuatorSerialNumber" value="v_e_019" />
+    <xacro:property name="leftAnkleRightActuatorSerialNumber" value="v_e_020" />
 	<xacro:property name="rightLegJ1SerialNumber" value="v_a_003" />
 	<xacro:property name="rightLegJ2SerialNumber" value="v_b_001" />
@@ -28,6 +28,6 @@
 	<xacro:property name="waistRightActuatorSerialNumber" value="v_e_005" />
 	<xacro:property name="waistLeftActuatorSerialNumber" value="v_e_006" />
-	<xacro:property name="leftForearmSerialNumber" value="v_h_001"/>
-        <xacro:property name="rightForearmSerialNumber" value="v_h_002"/>
+	<xacro:property name="leftForearmSerialNumber" value="v_h_007"/>
+    <xacro:property name="rightForearmSerialNumber" value="v_h_008"/>
 	<xacro:property name="left_foot_ATI_serial" value="FT16594" />
 	<xacro:property name="right_foot_ATI_serial" value="FT16592" />

File: common/xacro/serial_numbers/valkyrie_C_serials.xacro (robot description, xacro)
@@ -28,6 +28,6 @@
 	<xacro:property name="waistRightActuatorSerialNumber" value="v_e_014" />
 	<xacro:property name="waistLeftActuatorSerialNumber" value="v_e_013" />
-	<xacro:property name="leftForearmSerialNumber" value="v_h_007"/>
-        <xacro:property name="rightForearmSerialNumber" value="v_h_008"/>
+	<xacro:property name="leftForearmSerialNumber" value="v_h_001"/>
+    <xacro:property name="rightForearmSerialNumber" value="v_h_002"/>
 	<xacro:property name="left_foot_ATI_serial" value="FT14020" />
 	<xacro:property name="right_foot_ATI_serial" value="FT17214" />

Commit message: Swapped arm j5 serials.

File: common/xacro/serial_numbers/valkyrie_A_serials.xacro (robot description, xacro)
@@ -16,10 +16,10 @@
 	<xacro:property name="leftArmJ3SerialNumber" value="v_f_005" />
 	<xacro:property name="leftArmJ4SerialNumber" value="v_f_002" />
-	<xacro:property name="leftArmJ5SerialNumber" value="v_g_005" />
+	<xacro:property name="leftArmJ5SerialNumber" value="v_g_018" />
 	<xacro:property name="rightArmJ1SerialNumber" value="v_a_001" />
 	<xacro:property name="rightArmJ2SerialNumber" value="v_b_003" />
 	<xacro:property name="rightArmJ3SerialNumber" value="v_f_004" />
 	<xacro:property name="rightArmJ4SerialNumber" value="v_f_003" />
-	<xacro:property name="rightArmJ5SerialNumber" value="v_g_003" />
+	<xacro:property name="rightArmJ5SerialNumber" value="v_g_017" />
 	<xacro:property name="neckJ1SerialNumber" value="v_g_006" />
 	<xacro:property name="neckJ2SerialNumber" value="v_g_007" />

File: common/xacro/serial_numbers/valkyrie_C_serials.xacro (robot description, xacro)
@@ -16,10 +16,10 @@
 	<xacro:property name="leftArmJ3SerialNumber" value="v_f_012" />
 	<xacro:property name="leftArmJ4SerialNumber" value="v_f_011" />
-	<xacro:property name="leftArmJ5SerialNumber" value="v_g_018" />
+	<xacro:property name="leftArmJ5SerialNumber" value="v_g_005" />
 	<xacro:property name="rightArmJ1SerialNumber" value="v_a_012" />
 	<xacro:property name="rightArmJ2SerialNumber" value="v_b_012" />
 	<xacro:property name="rightArmJ3SerialNumber" value="v_f_013" />
 	<xacro:property name="rightArmJ4SerialNumber" value="v_f_014" />
-	<xacro:property name="rightArmJ5SerialNumber" value="v_g_017" />
+	<xacro:property name="rightArmJ5SerialNumber" value="v_g_003" />
 	<xacro:property name="neckJ1SerialNumber" value="v_g_001" />
 	<xacro:property name="neckJ2SerialNumber" value="v_g_002" />

Commit message: Switched the left leg coeffs between units A and B.

File: common/xacro/serial_numbers/valkyrie_A_serials.xacro (robot description, xacro)
@@ -1,9 +1,9 @@
 <robot xmlns:xacro="http://ros.org/wiki/xacro" name="valkyrie_A_serials">
 	<xacro:property name="leftLegJ1SerialNumber" value="v_a_006" />
-	<xacro:property name="leftLegJ2SerialNumber" value="v_b_006" />
-    <xacro:property name="leftLegJ3SerialNumber" value="v_c_004" />
-    <xacro:property name="leftLegJ4SerialNumber" value="v_d_003" />
-    <xacro:property name="leftAnkleLeftActuatorSerialNumber" value="v_e_019" />
-    <xacro:property name="leftAnkleRightActuatorSerialNumber" value="v_e_020" />
+	<xacro:property name="leftLegJ2SerialNumber" value="v_b_016" />
+	<xacro:property name="leftLegJ3SerialNumber" value="v_c_008" />
+	<xacro:property name="leftLegJ4SerialNumber" value="v_d_008" />
+	<xacro:property name="leftAnkleLeftActuatorSerialNumber" value="v_e_016" />
+	<xacro:property name="leftAnkleRightActuatorSerialNumber" value="v_e_015" />
 	<xacro:property name="rightLegJ1SerialNumber" value="v_a_003" />
 	<xacro:property name="rightLegJ2SerialNumber" value="v_b_001" />
@@ -30,5 +30,5 @@
 	<xacro:property name="leftForearmSerialNumber" value="v_h_007"/>
     <xacro:property name="rightForearmSerialNumber" value="v_h_008"/>
-	<xacro:property name="left_foot_ATI_serial" value="FT16594" />
+	<xacro:property name="left_foot_ATI_serial" value="FT17218" />
 	<xacro:property name="right_foot_ATI_serial" value="FT16592" />
 	<xacro:property name="sim_ATI_serial" value="FT001SIM" />

File: common/xacro/serial_numbers/valkyrie_B_serials.xacro (robot description, xacro)
@@ -1,9 +1,9 @@
 <robot xmlns:xacro="http://ros.org/wiki/xacro" name="valkyrie_B_serials">
 	<xacro:property name="leftLegJ1SerialNumber" value="v_a_009" />
-	<xacro:property name="leftLegJ2SerialNumber" value="v_b_016" />
-	<xacro:property name="leftLegJ3SerialNumber" value="v_c_008" />
-	<xacro:property name="leftLegJ4SerialNumber" value="v_d_008" />
-	<xacro:property name="leftAnkleLeftActuatorSerialNumber" value="v_e_016" />
-	<xacro:property name="leftAnkleRightActuatorSerialNumber" value="v_e_015" />
+	<xacro:property name="leftLegJ2SerialNumber" value="v_b_006" />
+    <xacro:property name="leftLegJ3SerialNumber" value="v_c_004" />
+    <xacro:property name="leftLegJ4SerialNumber" value="v_d_003" />
+    <xacro:property name="leftAnkleLeftActuatorSerialNumber" value="v_e_019" />
+    <xacro:property name="leftAnkleRightActuatorSerialNumber" value="v_e_020" />
 	<xacro:property name="rightLegJ1SerialNumber" value="v_a_007" />
 	<xacro:property name="rightLegJ2SerialNumber" value="v_b_015" />
@@ -30,5 +30,5 @@
 	<xacro:property name="leftForearmSerialNumber" value="v_h_003"/>
     <xacro:property name="rightForearmSerialNumber" value="v_h_004"/>
-	<xacro:property name="left_foot_ATI_serial" value="FT17218" />
+	<xacro:property name="left_foot_ATI_serial" value="FT16594" />
 	<xacro:property name="right_foot_ATI_serial" value="FT14018" />
     <xacro:property name="sim_ATI_serial" value="FT001SIM" />

Commit message: Moved ankle actuators and ATI from A back to B since we put the lower leg back on unit B that we took off earlier.

File: common/xacro/serial_numbers/valkyrie_A_serials.xacro (robot description, xacro)
@@ -4,6 +4,6 @@
 	<xacro:property name="leftLegJ3SerialNumber" value="v_c_008" />
 	<xacro:property name="leftLegJ4SerialNumber" value="v_d_008" />
-	<xacro:property name="leftAnkleLeftActuatorSerialNumber" value="v_e_016" />
-	<xacro:property name="leftAnkleRightActuatorSerialNumber" value="v_e_015" />
+	<xacro:property name="leftAnkleLeftActuatorSerialNumber" value="v_e_019" />
+    <xacro:property name="leftAnkleRightActuatorSerialNumber" value="v_e_020" />
 	<xacro:property name="rightLegJ1SerialNumber" value="v_a_003" />
 	<xacro:property name="rightLegJ2SerialNumber" value="v_b_001" />
@@ -30,5 +30,5 @@
 	<xacro:property name="leftForearmSerialNumber" value="v_h_007"/>
     <xacro:property name="rightForearmSerialNumber" value="v_h_008"/>
-	<xacro:property name="left_foot_ATI_serial" value="FT17218" />
+	<xacro:property name="left_foot_ATI_serial" value="FT16594" />
 	<xacro:property name="right_foot_ATI_serial" value="FT16592" />
 	<xacro:property name="sim_ATI_serial" value="FT001SIM" />

File: common/xacro/serial_numbers/valkyrie_B_serials.xacro (robot description, xacro)
@@ -4,6 +4,6 @@
     <xacro:property name="leftLegJ3SerialNumber" value="v_c_004" />
     <xacro:property name="leftLegJ4SerialNumber" value="v_d_003" />
-    <xacro:property name="leftAnkleLeftActuatorSerialNumber" value="v_e_019" />
-    <xacro:property name="leftAnkleRightActuatorSerialNumber" value="v_e_020" />
+	<xacro:property name="leftAnkleLeftActuatorSerialNumber" value="v_e_016" />
+	<xacro:property name="leftAnkleRightActuatorSerialNumber" value="v_e_015" />
 	<xacro:property name="rightLegJ1SerialNumber" value="v_a_007" />
 	<xacro:property name="rightLegJ2SerialNumber" value="v_b_015" />
@@ -30,5 +30,5 @@
 	<xacro:property name="leftForearmSerialNumber" value="v_h_003"/>
     <xacro:property name="rightForearmSerialNumber" value="v_h_004"/>
-	<xacro:property name="left_foot_ATI_serial" value="FT16594" />
+	<xacro:property name="left_foot_ATI_serial" value="FT17218" />
 	<xacro:property name="right_foot_ATI_serial" value="FT14018" />
     <xacro:property name="sim_ATI_serial" value="FT001SIM" />

Commit message: leg swapping and serial number shuffling. Losing track.

File: common/xacro/serial_numbers/valkyrie_A_serials.xacro (robot description, xacro)
@@ -1,9 +1,9 @@
 <robot xmlns:xacro="http://ros.org/wiki/xacro" name="valkyrie_A_serials">
 	<xacro:property name="leftLegJ1SerialNumber" value="v_a_006" />
-	<xacro:property name="leftLegJ2SerialNumber" value="v_b_016" />
-	<xacro:property name="leftLegJ3SerialNumber" value="v_c_008" />
-	<xacro:property name="leftLegJ4SerialNumber" value="v_d_008" />
-	<xacro:property name="leftAnkleLeftActuatorSerialNumber" value="v_e_019" />
-    <xacro:property name="leftAnkleRightActuatorSerialNumber" value="v_e_020" />
+	<xacro:property name="leftLegJ2SerialNumber" value="v_b_006" />
+    <xacro:property name="leftLegJ3SerialNumber" value="v_c_004" />
+    <xacro:property name="leftLegJ4SerialNumber" value="v_d_003" />
+    <xacro:property name="leftAnkleLeftActuatorSerialNumber" value="v_e_016" />
+	<xacro:property name="leftAnkleRightActuatorSerialNumber" value="v_e_015" />
 	<xacro:property name="rightLegJ1SerialNumber" value="v_a_003" />
 	<xacro:property name="rightLegJ2SerialNumber" value="v_b_001" />

File: common/xacro/serial_numbers/valkyrie_B_serials.xacro (robot description, xacro)
@@ -1,9 +1,9 @@
 <robot xmlns:xacro="http://ros.org/wiki/xacro" name="valkyrie_B_serials">
 	<xacro:property name="leftLegJ1SerialNumber" value="v_a_009" />
-	<xacro:property name="leftLegJ2SerialNumber" value="v_b_006" />
-    <xacro:property name="leftLegJ3SerialNumber" value="v_c_004" />
-    <xacro:property name="leftLegJ4SerialNumber" value="v_d_003" />
-	<xacro:property name="leftAnkleLeftActuatorSerialNumber" value="v_e_016" />
-	<xacro:property name="leftAnkleRightActuatorSerialNumber" value="v_e_015" />
+    <xacro:property name="leftLegJ2SerialNumber" value="v_b_016" />
+	<xacro:property name="leftLegJ3SerialNumber" value="v_c_008" />
+	<xacro:property name="leftLegJ4SerialNumber" value="v_d_008" />
+	<xacro:property name="leftAnkleLeftActuatorSerialNumber" value="v_e_019" />
+    <xacro:property name="leftAnkleRightActuatorSerialNumber" value="v_e_020" />
 	<xacro:property name="rightLegJ1SerialNumber" value="v_a_007" />
 	<xacro:property name="rightLegJ2SerialNumber" value="v_b_015" />

Commit message: swapped ATI serials.

File: common/xacro/serial_numbers/valkyrie_A_serials.xacro (robot description, xacro)
@@ -30,5 +30,5 @@
 	<xacro:property name="leftForearmSerialNumber" value="v_h_007"/>
     <xacro:property name="rightForearmSerialNumber" value="v_h_008"/>
-	<xacro:property name="left_foot_ATI_serial" value="FT16594" />
+	<xacro:property name="left_foot_ATI_serial" value="FT17218" />
 	<xacro:property name="right_foot_ATI_serial" value="FT16592" />
 	<xacro:property name="sim_ATI_serial" value="FT001SIM" />

File: common/xacro/serial_numbers/valkyrie_B_serials.xacro (robot description, xacro)
@@ -30,5 +30,5 @@
 	<xacro:property name="leftForearmSerialNumber" value="v_h_003"/>
     <xacro:property name="rightForearmSerialNumber" value="v_h_004"/>
-	<xacro:property name="left_foot_ATI_serial" value="FT17218" />
+	<xacro:property name="left_foot_ATI_serial" value="FT16594" />
 	<xacro:property name="right_foot_ATI_serial" value="FT14018" />
     <xacro:property name="sim_ATI_serial" value="FT001SIM" />
