Commit message: Put new IMU on unit B. Calibrated unit B legs.

File: common/xacro/dev_ports/valkyrie_B_ports.xacro (robot description, xacro)
@@ -2,5 +2,6 @@
 	<xacro:property name="pelvis_middle_imu_port" value="/dev/serial/by-id/usb-Lord_Microstrain_Lord_Inertial_Sensor_0000__6233.47094-if00" />
 	<!-- <xacro:property name="pelvis_rear_imu_port" value="/dev/serial/by-id/usb-FTDI_USB-RS232_Cable_FTY5H9NH-if00-port0" /> -->
-        <xacro:property name="pelvis_rear_imu_port" value="/dev/serial/by-id/usb-Lord_Microstrain_Lord_Inertial_Sensor_0000__6233.47099-if00" />
+  <!-- <xacro:property name="pelvis_rear_imu_port" value="/dev/serial/by-id/usb-Lord_Microstrain_Lord_Inertial_Sensor_0000__6233.47099-if00" /> -->
+  <xacro:property name="pelvis_rear_imu_port" value="/dev/serial/by-id/usb-Lord_Microstrain_Lord_Inertial_Sensor_0000__6233.47092-if00" />
 	<xacro:property name="torso_left_imu_port" value="/dev/serial/by-id/usb-Lord_Microstrain_Lord_Inertial_Sensor_0000__6233.47097-if00" />
 </robot>
