Commit message: Changes to at least compile under ROS distributions > Jade. Tested on Melodic. Files are missing, and the URDF files was forced in the repo taken by IHMC

File: common/xacro/actuator_names/valkyrie_actuator_names.xacro (robot description, xacro)
@@ -1,4 +1,4 @@
 <?xml version="1.0" ?>
-<robot name="valkyrie_joint_names" xmlns:xacro="http://www.ros.org/wiki/xacro">
+<robot name="valkyrie_joint_names" xmlns:xacro="http://wiki.ros.org/xacro">
 	<xacro:property name="TorsoYawActuatorName" value="torsoYaw"/>
 	<xacro:property name="WaistLeftActuatorName" value="waistLeftActuator"/>

File: common/xacro/api/valkyrie_api.xacro (robot description, xacro)
@@ -1,3 +1,3 @@
-<robot xmlns:xacro="http://ros.org/wiki/xacro" name="valkyrie_api">
+<robot xmlns:xacro="http://wiki.ros.org/xacro" name="valkyrie_api">
 	<xacro:property name="HipYawApi" value="robot_hardware_interface/TurbodriverAPI_DRCv4" />
 	<xacro:property name="HipRollApi" value="robot_hardware_interface/TurbodriverAPI_DRCv4" />

File: common/xacro/joint_names/valkyrie_joint_names.xacro (robot description, xacro)
@@ -1,4 +1,4 @@
 <?xml version="1.0" ?>
-<robot name="valkyrie_joint_names" xmlns:xacro="http://www.ros.org/wiki/xacro">
+<robot name="valkyrie_joint_names" xmlns:xacro="http://wiki.ros.org/xacro">
 	<xacro:property name="TorsoYawJointName" value="torsoYaw"/>
 	<xacro:property name="TorsoPitchJointName" value="torsoPitch"/>

File: common/xacro/nodes/test_bench_nodes.xacro (robot description, xacro)
@@ -1,3 +1,3 @@
-<robot xmlns:xacro="http://ros.org/wiki/xacro" name="valkyrie_nodes">
+<robot xmlns:xacro="http://wiki.ros.org/xacro" name="valkyrie_nodes">
 	<xacro:property name="testbench_node" value="/left_arm/j0" />
 </robot>

File: common/xacro/nodes/valkyrie_nodes.xacro (robot description, xacro)
@@ -1,3 +1,3 @@
-<robot xmlns:xacro="http://ros.org/wiki/xacro" name="valkyrie_nodes">
+<robot xmlns:xacro="http://wiki.ros.org/xacro" name="valkyrie_nodes">
 	<xacro:property name="HipYawNode" value="/pelvis/${prefix}_leg_j1" />
 	<xacro:property name="HipRollNode" value="/${prefix}_leg/j2" />
@@ -17,20 +17,5 @@
 	<xacro:property name="WristRollActuatorSimNode" value="/${prefix}_arm/wrist/roll_actautor" />
 	<xacro:property name="WristPitchActuatorSimNode" value="/${prefix}_arm/wrist/pitch_actuator" />
-	<xacro:property name="LowerNeckPitchNode" value="/neck/j1" />
-	<xacro:property name="NeckYawNode" value="/neck/j2" />
-	<xacro:property name="UpperNeckPitchNode" value="/neck/j3" />
-	<xacro:property name="TrunkYawNode" value="/pelvis/waist" /> <!--Yaw-->
-	<xacro:property name="WaistLeftActuatorNode" value="/trunk/left_actuator" /> <!--pitch-->
-	<xacro:property name="WaistRightActuatorNode" value="/trunk/right_actuator" /> <!--roll-->
-	<xacro:property name="WaistPitchActuatorSimNode" value="/trunk/pitch_actuator" /> <!--pitch-->
-	<xacro:property name="WaistRollActuatorSimNode" value="/trunk/roll_actuator" /> <!--roll-->
-	<xacro:property name="pelvis_imu1_node" value="/pelvis/sensors/imu1" />
-	<xacro:property name="pelvis_imu2_node" value="/pelvis/sensors/imu2" />
-	<xacro:property name="torso_imu1_node" value="/torso/sensors/imu1" />
-	<xacro:property name="torso_imu2_node" value="/torso/sensors/imu2" />
-	<xacro:property name="left_foot_ATI_node" value="/left_leg/ankle/left_actuator" />
-	<xacro:property name="left_foot_Sim_ATI_node" value="/sensors/leftFootSixAxis" />
-	<xacro:property name="right_foot_ATI_node" value="/right_leg/ankle/left_actuator" />
-	<xacro:property name="right_foot_Sim_ATI_node" value="/sensors/rightFootSixAxis" />
+	<xacro:include filename="$(find val_description)/common/xacro/nodes/regular_nodes.xacro" />
 	<xacro:macro name="all_channels" >
 		<Channels>

File: common/xacro/serial_numbers/test_bench_serials.xacro (robot description, xacro)
@@ -1,3 +1,3 @@
-<robot xmlns:xacro="http://ros.org/wiki/xacro" name="test_bench_serials">
+<robot xmlns:xacro="http://wiki.ros.org/xacro" name="test_bench_serials">
 	<xacro:property name="testbench_serial_number" value="v_a_013" />
 </robot>

File: common/xacro/serial_numbers/valkyrie_A_serials.xacro (robot description, xacro)
@@ -1,3 +1,3 @@
-<robot xmlns:xacro="http://ros.org/wiki/xacro" name="valkyrie_A_serials">
+<robot xmlns:xacro="http://wiki.ros.org/xacro" name="valkyrie_A_serials">
 	<xacro:property name="leftLegJ1SerialNumber" value="v_a_006" />
 	<xacro:property name="leftLegJ2SerialNumber" value="v_b_002" />

File: common/xacro/serial_numbers/valkyrie_B_serials.xacro (robot description, xacro)
@@ -1,3 +1,3 @@
-<robot xmlns:xacro="http://ros.org/wiki/xacro" name="valkyrie_B_serials">
+<robot xmlns:xacro="http://wiki.ros.org/xacro" name="valkyrie_B_serials">
 	<xacro:property name="leftLegJ1SerialNumber" value="v_a_009" />
 	<xacro:property name="leftLegJ2SerialNumber" value="v_b_006" />

File: common/xacro/serial_numbers/valkyrie_C_serials.xacro (robot description, xacro)
@@ -1,3 +1,3 @@
-<robot xmlns:xacro="http://ros.org/wiki/xacro" name="valkyrie_C_serials">
+<robot xmlns:xacro="http://wiki.ros.org/xacro" name="valkyrie_C_serials">
 	<xacro:property name="leftLegJ1SerialNumber" value="v_a_015" />
 	<xacro:property name="leftLegJ2SerialNumber" value="v_b_011" />

File: instance/instances/robots/test_bench.xacro (robot description, xacro)
@@ -1,3 +1,3 @@
-<robot xmlns:xacro="http://ros.org/wiki/xacro" name="testbench">
+<robot xmlns:xacro="http://wiki.ros.org/xacro" name="testbench">
 	<xacro:property name="instance" value="testbench" />
     <xacro:include filename="xacro/common/test_bench_template.xacro"/>

File: instance/instances/robots/valkyrie_A.xacro (robot description, xacro)
@@ -1,3 +1,3 @@
-<robot xmlns:xacro="http://ros.org/wiki/xacro" name="valkyrie_A">
+<robot xmlns:xacro="http://wiki.ros.org/xacro" name="valkyrie_A">
 	<xacro:property name="instance" value="valkyrie_A" />
 	<xacro:include filename="$(find val_description)/common/xacro/serial_numbers/valkyrie_A_serials.xacro" />

File: instance/instances/robots/valkyrie_B.xacro (robot description, xacro)
@@ -1,3 +1,3 @@
-<robot xmlns:xacro="http://ros.org/wiki/xacro" name="valkyrie_B">
+<robot xmlns:xacro="http://wiki.ros.org/xacro" name="valkyrie_B">
 	<xacro:property name="instance" value="valkyrie_B" />
 	<xacro:include filename="$(find val_description)/common/xacro/serial_numbers/valkyrie_B_serials.xacro" />

File: instance/instances/robots/valkyrie_C.xacro (robot description, xacro)
@@ -1,3 +1,3 @@
-<robot xmlns:xacro="http://ros.org/wiki/xacro" name="valkyrie_C">
+<robot xmlns:xacro="http://wiki.ros.org/xacro" name="valkyrie_C">
 	<xacro:property name="instance" value="valkyrie_C" />
 	<xacro:include filename="$(find val_description)/common/xacro/serial_numbers/valkyrie_C_serials.xacro" />

File: instance/instances/robots/xacro/common/test_bench_template.xacro (robot description, xacro)
@@ -1,3 +1,3 @@
-<robot xmlns:xacro="http://ros.org/wiki/xacro" name="test_bench_template">
+<robot xmlns:xacro="http://wiki.ros.org/xacro" name="test_bench_template">
 	<xacro:include filename="$(find val_description)/common/xacro/serial_numbers/test_bench_serials.xacro" />
 	<xacro:include filename="$(find val_description)/common/xacro/nodes/test_bench_nodes.xacro" />

File: instance/instances/robots/xacro/common/valkyrie_full_template.xacro (robot description, xacro)
@@ -1,4 +1,4 @@
-<robot xmlns:xacro="http://ros.org/wiki/xacro" name="valkyrie_template">
-	<xacro:include filename="$(find val_description)/common/xacro/nodes/valkyrie_nodes.xacro" />
+<robot xmlns:xacro="http://wiki.ros.org/xacro" name="valkyrie_template">
+	<xacro:include filename="$(find val_description)/common/xacro/nodes/regular_nodes.xacro" />
 	<xacro:include filename="$(find val_description)/instance/instances/robots/xacro/limbs/leg.xacro" />
 	<xacro:include filename="$(find val_description)/instance/instances/robots/xacro/limbs/arm.xacro" />

File: instance/instances/robots/xacro/devices/devices.xacro (robot description, xacro)
@@ -1,3 +1,3 @@
-<robot xmlns:xacro="http://ros.org/wiki/xacro" name="actuators">
+<robot xmlns:xacro="http://wiki.ros.org/xacro" name="actuators">
   <xacro:macro name="imu" params="name serial_number node">
   	<Device id="${name}" type="imu">

File: instance/instances/robots/xacro/limbs/arm.xacro (robot description, xacro)
@@ -1,6 +1,7 @@
-<robot xmlns:xacro="http://ros.org/wiki/xacro" name="arm">
+<robot xmlns:xacro="http://wiki.ros.org/xacro" name="arm">
     <xacro:include filename="$(find val_description)/instance/instances/robots/xacro/mechanisms/mechanisms.xacro"/>
-    <xacro:include filename="$(find val_description)/common/xacro/joint_names/valkyrie_joint_names.xacro"/>
     <xacro:macro name="arm" params="prefix j1_serial_number j2_serial_number j3_serial_number j4_serial_number j5_serial_number wrist_actuator0_serial wrist_actuator1_serial" >
+        <xacro:include filename="$(find val_description)/common/xacro/nodes/valkyrie_nodes.xacro" />
+        <xacro:include filename="$(find val_description)/common/xacro/joint_names/valkyrie_joint_names.xacro"/>
     	<xacro:simple_mechanism name="${ShoulderPitchJointName}" serial_number="${j1_serial_number}" node="${ShoulderPitchNode}"/>
     	<xacro:simple_mechanism name="${ShoulderRollJointName}" serial_number="${j2_serial_number}" node="${ShoulderRollNode}"/>

File: instance/instances/robots/xacro/limbs/leg.xacro (robot description, xacro)
@@ -1,7 +1,8 @@
-<robot xmlns:xacro="http://ros.org/wiki/xacro" name="leg">
+<robot xmlns:xacro="http://wiki.ros.org/xacro" name="leg">
     <xacro:include filename="$(find val_description)/instance/instances/robots/xacro/mechanisms/mechanisms.xacro"/>
-    <xacro:include filename="$(find val_description)/common/xacro/joint_names/valkyrie_joint_names.xacro"/>
     <xacro:macro name="leg" params="prefix j1_serial_number j2_serial_number j3_serial_number j4_serial_number ankle_left_actuator_serial ankle_right_actuator_serial" >
-    	<xacro:simple_mechanism name="${HipYawJointName}" serial_number="${j1_serial_number}" node="${HipYawNode}"/>
+        <xacro:include filename="$(find val_description)/common/xacro/nodes/valkyrie_nodes.xacro" />
+        <xacro:include filename="$(find val_description)/common/xacro/joint_names/valkyrie_joint_names.xacro"/>
+        <xacro:simple_mechanism name="${HipYawJointName}" serial_number="${j1_serial_number}" node="${HipYawNode}"/>
     	<xacro:simple_mechanism name="${HipRollJointName}" serial_number="${j2_serial_number}" node="${HipRollNode}"/>
     	<xacro:simple_mechanism name="${HipPitchJointName}" serial_number="${j3_serial_number}" node="${HipPitchNode}"/>

File: instance/instances/robots/xacro/limbs/neck.xacro (robot description, xacro)
@@ -1,3 +1,3 @@
-<robot xmlns:xacro="http://ros.org/wiki/xacro" name="neck">
+<robot xmlns:xacro="http://wiki.ros.org/xacro" name="neck">
     <xacro:include filename="$(find val_description)/instance/instances/robots/xacro/mechanisms/mechanisms.xacro"/>
     <xacro:include filename="$(find val_description)/common/xacro/joint_names/valkyrie_joint_names.xacro"/>

File: instance/instances/robots/xacro/limbs/waist.xacro (robot description, xacro)
@@ -1,4 +1,4 @@
-<robot xmlns:xacro="http://ros.org/wiki/xacro" name="waist">
-    <xacro:include filename="xacro/mechanisms/mechanisms.xacro"/>
+<robot xmlns:xacro="http://wiki.ros.org/xacro" name="waist">
+    <xacro:include filename="../mechanisms/mechanisms.xacro"/>
     <xacro:macro name="waist" params="j1_serial_number waist_left_actuator_serial waist_right_actuator_serial" >
     	<xacro:simple_mechanism name="torso_yaw" serial_number="${j1_serial_number}" node="${TrunkYawNode}"/>
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